Commit message: finalising ver1

File: workspace/src/robot_sim/urdf/robot.urdf (robot description, URDF)
Before this commit: robot diffbot, 3 links, 2 joints
Links:
- added link front_caster; visual sphere radius=0.04
- link base_link: mass 5 -> None; geometry visual box size=0.4 0.3 0.1
- link left_wheel: mass 1 -> None; geometry visual cylinder length=0.04 radius=0.05
- link right_wheel: mass 1 -> None; geometry visual cylinder length=0.04 radius=0.05
Joints:
- added joint caster_joint: type fixed, parent base_link, child front_caster, origin xyz=0.2 0 -0.05
- joint left_wheel_joint: axis 0 1 0 -> (none); origin xyz=0 0.25 0 -> xyz=0 0.15 -0.05 rpy=0 1.57 0; type continuous -> fixed
- joint right_wheel_joint: axis 0 1 0 -> (none); origin xyz=0 -0.25 0 -> xyz=0 -0.15 -0.05 rpy=0 1.57 0; type continuous -> fixed
